File: hardware/kim-1-programmable-memory.kicad_sch (KiCad schematic)
At the start: 44 parts, among them J1 Conn_02x01, J2 EDGE_CONN, J3 VGA, J4 VIdeo Out, J5 Micro_SD_Card_Det1, Q1 DMG2305UX, SW1 RESET, U1 LVC04, U2 74LVC1G38, U3 74LVC541, U4 74LVC541, U5 74LVC245, U6 74LVC1G27, U7 LVC04, U8 PicoW

Commit message: Minor silkscreen changes, track width corrections, open hole for Pico antenna
Parts:
- C1, C11, C2, C4, C5, C6, C7: LCSC C77055 -> C14663
- C10: LCSC C344022 -> C96446
- C3: LCSC C77055 -> (none); MPN (none) -> C14663
- C8: LCSC C77082 -> C28233
- D1: LCSC C497932 -> C2286
- J1, J3, U8: now fitted; now in the parts list
- J2: footprint MTU_Library:EDGE_CONN -> MTU:EDGE_CONN; now fitted
- R1, R2, R3: LCSC C25995 -> C22978
- R10, R11, R8, R9: value 40R -> 47R; LCSC C23047 -> C23182
- R19: LCSC C159890 -> C22775
- R4, R7: LCSC C15401 -> C25804
- U7: footprint Package_SO:SOIC-14_3.9x8.7mm_P1.27mm -> SOIC:SOIC-14_3.9x8.7mm_P1.27mm
Changed lines of the file:
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@@
       (effects (font (size 1.27 1.27)) hide)
     )
-    (property "LCSC" "C77055" (at 58.42 165.1 90)
+    (property "LCSC" "C14663" (at 58.42 165.1 90)
       (effects (font (size 1.27 1.27)) hide)
     )
@@
       (effects (font (size 1.27 1.27)) hide)
     )
-    (property "LCSC" "C77055" (at 57.15 266.7 90)
+    (property "LCSC" "C14663" (at 57.15 266.7 90)
       (effects (font (size 1.27 1.27)) hide)
     )
@@
       (effects (font (size 1.27 1.27)) (justify right))
     )
-    (property "Value" "40R" (at 176.53 171.45 90)
+    (property "Value" "47R" (at 176.53 171.45 90)
       (effects (font (size 1.27 1.27)) (justify right))
     )
@@
       (effects (font (size 1.27 1.27)) hide)
     )
-    (property "LCSC" "C23047" (at 176.53 168.91 90)
+    (property "LCSC" "C23182" (at 176.53 168.91 90)
       (effects (font (size 1.27 1.27)) hide)
     )
@@
       (effects (font (size 1.27 1.27)) hide)
     )
-    (property "LCSC" "C25995" (at 97.79 210.82 0)
+    (property "LCSC" "C22978" (at 97.79 210.82 0)
       (effects (font (size 1.27 1.27)) hide)
     )
@@
       (effects (font (size 1.27 1.27)) hide)
     )
-    (property "LCSC" "C159890" (at 213.995 139.7 90)
+    (property "LCSC" "C22775" (at 213.995 139.7 90)
       (effects (font (size 1.27 1.27)) hide)
     )
@@
   )
   (symbol (lib_id "Connector_Generic:Conn_02x01") (at 33.02 278.13 0) (unit 1)
-    (in_bom no) (on_board yes) (dnp yes) (fields_autoplaced)
+    (in_bom yes) (on_board yes) (dnp no) (fields_autoplaced)
     (property "Reference" "J1" (at 34.29 274.32 0)
       (effects (font (size 1.27 1.27)))
@@
       (effects (font (size 1.27 1.27)) hide)
     )
-    (property "LCSC" "C497932" (at 205.105 139.7 0)
+    (property "LCSC" "C2286" (at 205.105 139.7 0)
       (effects (font (size 1.27 1.27)) hide)
     )
@@
   )
   (symbol (lib_id "PicoW:PicoW") (at 220.98 95.885 0) (unit 1)
-    (in_bom no) (on_board yes) (dnp yes) (fields_autoplaced)
+    (in_bom yes) (on_board yes) (dnp no) (fields_autoplaced)
     (property "Reference" "U8" (at 220.98 64.135 0)
       (effects (font (size 1.27 1.27)))
@@
       (effects (font (size 1.27 1.27)) hide)
     )
-    (property "LCSC" "C25995" (at 107.95 153.67 0)
+    (property "LCSC" "C22978" (at 107.95 153.67 0)
       (effects (font (size 1.27 1.27)) hide)
     )
@@
   )
   (symbol (lib_id "Connector:DA15_Receptacle_MountingHoles") (at 180.34 247.015 0) (mirror y) (unit 1)
-    (in_bom no) (on_board yes) (dnp yes)
+    (in_bom yes) (on_board yes) (dnp no)
     (property "Reference" "J3" (at 180.34 222.885 0)
       (effects (font (size 1.27 1.27)))
@@
       (effects (font (size 1.27 1.27)) hide)
     )
-    (property "LCSC" "C15401" (at 208.915 161.29 0)
+    (property "LCSC" "C25804" (at 208.915 161.29 0)
       (effects (font (size 1.27 1.27)) hide)
     )
@@
       (effects (font (size 1.27 1.27)) hide)
     )
-    (property "LCSC" "C77055" (at 87.63 259.08 90)
+    (property "LCSC" "C14663" (at 87.63 259.08 90)
       (effects (font (size 1.27 1.27)) hide)
     )
@@
       (effects (font (size 1.27 1.27)) hide)
     )
-    (property "LCSC" "C77055" (at 194.945 311.15 0)
+    (property "LCSC" "C14663" (at 194.945 311.15 0)
       (effects (font (size 1.27 1.27)) hide)
     )
@@
       (effects (font (size 1.27 1.27)) (justify left))
     )
-    (property "Footprint" "Package_SO:SOIC-14_3.9x8.7mm_P1.27mm" (at 211.455 321.31 0)
+    (property "Footprint" "SOIC:SOIC-14_3.9x8.7mm_P1.27mm" (at 211.455 321.31 0)
       (effects (font (size 1.27 1.27)) hide)
     )
@@
       (effects (font (size 1.27 1.27)) hide)
     )
-    (property "LCSC" "C77055" (at 58.42 106.68 90)
+    (property "LCSC" "C14663" (at 58.42 106.68 90)
       (effects (font (size 1.27 1.27)) hide)
     )
@@
       (effects (font (size 1.27 1.27)) (justify right))
     )
-    (property "Value" "40R" (at 210.82 181.61 90)
+    (property "Value" "47R" (at 210.82 181.61 90)
       (effects (font (size 1.27 1.27)) (justify right))
     )
@@
       (effects (font (size 1.27 1.27)) hide)
     )
-    (property "LCSC" "C23047" (at 210.82 179.07 90)
+    (property "LCSC" "C23182" (at 210.82 179.07 90)
       (effects (font (size 1.27 1.27)) hide)
     )
@@
       (effects (font (size 1.27 1.27)) hide)
     )
-    (property "LCSC" "C77055" (at 202.565 190.5 0)
+    (property "LCSC" "C14663" (at 202.565 190.5 0)
       (effects (font (size 1.27 1.27)) hide)
     )
@@
       (effects (font (size 1.27 1.27)) hide)
     )
-    (property "LCSC" "C25995" (at 46.99 274.32 0)
+    (property "LCSC" "C22978" (at 46.99 274.32 0)
       (effects (font (size 1.27 1.27)) hide)
     )
@@
       (effects (font (size 1.27 1.27)) (justify left))
     )
-    (property "Footprint" "Package_SO:SOIC-14_3.9x8.7mm_P1.27mm" (at 234.315 219.075 0)
+    (property "Footprint" "SOIC:SOIC-14_3.9x8.7mm_P1.27mm" (at 234.315 219.075 0)
       (effects (font (size 1.27 1.27)) hide)
     )
@@
       (effects (font (size 1.27 1.27)) (justify left))
     )
-    (property "Footprint" "Package_SO:SOIC-14_3.9x8.7mm_P1.27mm" (at 234.315 239.395 0)
+    (property "Footprint" "SOIC:SOIC-14_3.9x8.7mm_P1.27mm" (at 234.315 239.395 0)
       (effects (font (size 1.27 1.27)) hide)
     )
@@
       (effects (font (size 1.27 1.27)) hide)
     )
-    (property "LCSC" "C77055" (at 58.42 48.26 90)
+    (property "MPN" "C14663" (at 58.42 48.26 90)
       (effects (font (size 1.27 1.27)) hide)
     )
@@
       (effects (font (size 1.27 1.27)) hide)
     )
-    (property "LCSC" "C15401" (at 189.23 161.29 0)
+    (property "LCSC" "C25804" (at 189.23 161.29 0)
       (effects (font (size 1.27 1.27)) hide)
     )
@@
       (effects (font (size 1.27 1.27)))
     )
-    (property "Footprint" "Package_SO:SOIC-14_3.9x8.7mm_P1.27mm" (at 234.315 259.08 0)
+    (property "Footprint" "SOIC:SOIC-14_3.9x8.7mm_P1.27mm" (at 234.315 259.08 0)
       (effects (font (size 1.27 1.27)) hide)
     )
@@
       (effects (font (size 1.27 1.27)) (justify right))
     )
-    (property "Value" "40R" (at 176.53 163.83 90)
+    (property "Value" "47R" (at 176.53 163.83 90)
       (effects (font (size 1.27 1.27)) (justify right))
     )
@@
       (effects (font (size 1.27 1.27)) hide)
     )
-    (property "LCSC" "C23047" (at 176.53 166.37 90)
+    (property "LCSC" "C23182" (at 176.53 166.37 90)
       (effects (font (size 1.27 1.27)) hide)
     )
@@
       (effects (font (size 1.27 1.27)) (justify left))
     )
-    (property "Footprint" "Package_SO:SOIC-14_3.9x8.7mm_P1.27mm" (at 234.315 208.915 0)
+    (property "Footprint" "SOIC:SOIC-14_3.9x8.7mm_P1.27mm" (at 234.315 208.915 0)
       (effects (font (size 1.27 1.27)) hide)
     )
@@
       (effects (font (size 1.27 1.27)) (justify left))
     )
-    (property "Footprint" "Package_SO:SOIC-14_3.9x8.7mm_P1.27mm" (at 234.315 248.92 0)
+    (property "Footprint" "SOIC:SOIC-14_3.9x8.7mm_P1.27mm" (at 234.315 248.92 0)
       (effects (font (size 1.27 1.27)) hide)
     )
@@
       (effects (font (size 1.27 1.27)) hide)
     )
-    (property "LCSC" "C77082" (at 148.59 319.405 0)
+    (property "LCSC" "C28233" (at 148.59 319.405 0)
       (effects (font (size 1.27 1.27)) hide)
     )
@@
       (effects (font (size 1.27 1.27)) hide)
     )
-    (property "LCSC" "C77055" (at 220.98 311.15 0)
+    (property "LCSC" "C14663" (at 220.98 311.15 0)
       (effects (font (size 1.27 1.27)) hide)
     )
@@
   )
   (symbol (lib_id "MTU_Library:EDGE_CONN") (at 88.9 324.485 270) (unit 1)
-    (in_bom no) (on_board yes) (dnp yes) (fields_autoplaced)
+    (in_bom no) (on_board yes) (dnp no) (fields_autoplaced)
     (property "Reference" "J2" (at 87.63 342.265 90)
       (effects (font (size 1.27 1.27)))
@@
       (effects (font (size 1.27 1.27)))
     )
-    (property "Footprint" "MTU_Library:EDGE_CONN" (at 88.9 321.31 0)
+    (property "Footprint" "MTU:EDGE_CONN" (at 88.9 321.31 0)
       (effects (font (size 1.27 1.27)) hide)
     )
@@
       (effects (font (size 1.27 1.27)) (justify left))
     )
-    (property "Footprint" "Package_SO:SOIC-14_3.9x8.7mm_P1.27mm" (at 234.315 229.235 0)
+    (property "Footprint" "SOIC:SOIC-14_3.9x8.7mm_P1.27mm" (at 234.315 229.235 0)
       (effects (font (size 1.27 1.27)) hide)
     )
@@
       (effects (font (size 1.27 1.27)) hide)
     )
-    (property "LCSC" "C344022" (at 196.215 190.5 0)
+    (property "LCSC" "C96446" (at 196.215 190.5 0)
       (effects (font (size 1.27 1.27)) hide)
     )
@@
       (effects (font (size 1.27 1.27)) (justify right))
     )
-    (property "Value" "40R" (at 176.53 176.53 90)
+    (property "Value" "47R" (at 176.53 176.53 90)
       (effects (font (size 1.27 1.27)) (justify right))
     )
@@
       (effects (font (size 1.27 1.27)) hide)
     )
-    (property "LCSC" "C23047" (at 176.53 173.99 90)
-      (effects (font (size 1.27 1.27)) hide)
-    )
+    (property "LCSC" "C23182" (at 176.53 173.99 90)
+      (effects (font (size 1.27 1.27)) hide)
+    )

Commit message: New design: bus multiplexing and video and sd card support
Parts:
- R19: value 100R -> 150R
Connections:
- net GND: now also U4.1 (G1); no longer U3.1 (G1)
- net at R3.1, U1.2: now also U3.1 (G1); no longer U4.1 (G1)
Changed lines of the file:
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@@
   (junction (at 133.35 214.63) (diameter 0) (color 0 0 0 0)
   )
+  (junction (at 49.53 140.97) (diameter 0) (color 0 0 0 0)
+  )
   (junction (at 185.42 307.34) (diameter 0) (color 0 0 0 0)
   )
@@
   )
   (junction (at 211.455 307.34) (diameter 0) (color 0 0 0 0)
-  )
-  (junction (at 49.53 82.55) (diameter 0) (color 0 0 0 0)
   )
   (junction (at 191.135 254.635) (diameter 0) (color 0 0 0 0)
@@
     (stroke (width 0) (type default))
   )
-  (wire (pts (xy 52.07 138.43) (xy 46.99 138.43))
+  (wire (pts (xy 52.07 138.43) (xy 49.53 138.43))
     (stroke (width 0) (type default))
   )
@@
     (stroke (width 0) (type default))
   )
-  (wire (pts (xy 49.53 80.01) (xy 49.53 82.55))
+  (wire (pts (xy 46.99 80.01) (xy 46.99 157.48))
     (stroke (width 0) (type default))
   )
@@
     (stroke (width 0) (type default))
   )
-  (wire (pts (xy 52.07 80.01) (xy 49.53 80.01))
+  (wire (pts (xy 52.07 80.01) (xy 46.99 80.01))
     (stroke (width 0) (type default))
   )
@@
     (stroke (width 0) (type default))
   )
-  (wire (pts (xy 46.99 138.43) (xy 46.99 157.48))
-    (stroke (width 0) (type default))
-  )
   (bus (pts (xy 147.32 135.89) (xy 147.32 133.35))
     (stroke (width 0) (type default) (color 194 0 194 1))
@@
   )
   (bus (pts (xy 17.78 299.72) (xy 60.96 299.72))
+    (stroke (width 0) (type default))
+  )
+  (wire (pts (xy 49.53 138.43) (xy 49.53 140.97))
     (stroke (width 0) (type default))
   )
@@
       (effects (font (size 1.27 1.27)) (justify right))
     )
-    (property "Value" "100R" (at 216.535 142.24 90)
+    (property "Value" "150R" (at 216.535 142.24 90)
       (effects (font (size 1.27 1.27)) (justify right))
     )

Commit message: Silly silkscreen mistake
Parts:
- D1: value HDD -> FDC
Changed lines of the file:
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@@
       (effects (font (size 1.27 1.27)))
     )
-    (property "Value" "HDD" (at 205.105 142.875 0)
+    (property "Value" "FDC" (at 205.105 142.875 0)
       (effects (font (size 1.27 1.27)))
     )
